Commit message: modify end effector position

File: pkg_rp_arm/urdf/rp.urdf.xacro (robot description, xacro)
@@ -105,5 +105,5 @@
     </link>
     <joint name="slider_EE_joint" type="fixed">
-        <origin xyz="0 -0.08 0" rpy="1.55 0 0"/>
+        <origin xyz="0 0 -0.18" rpy="0 0 0"/>
         <parent link="slider_link"/>
         <child link="end_effector"/>

Commit message: fix end effector start point

File: pkg_rp_arm/urdf/rp.urdf.xacro (robot description, xacro)
@@ -84,9 +84,9 @@
     </link>
     <joint name="slider_joint" type="prismatic">
-        <origin xyz="0 0 0" rpy="0 0 0"/>
+        <origin xyz="-0.4 0 0" rpy="0 0 0"/>
         <parent link="rod_link"/>
         <child link="slider_link"/>
         <axis xyz="1 0 0"/>
-        <limit lower="0.6" upper="-0.6" velocity="100" effort="100"/>
+        <limit lower="0" upper="1.0" velocity="100" effort="100"/>
     </joint>
    <link name="slider_link">
